Commit message: 更新

File: sobit_description/robots/sobit.urdf (robot description, URDF)
Before this commit: robot sobit, 24 links, 23 joints
Links:
- link base_frame: geometry collision mesh filename=package://sobit_description/mesh/stl/SOBIT_MainFrame v1.stl; visual mesh filename=package://sobit_description/mesh/stl/SOBIT_MainFrame v1.stl
- link chin: geometry visual mesh filename=package://sobit_description/mesh/stl/SOBIT_chin.stl
- link head: geometry visual mesh filename=package://sobit_description/mesh/stl/SOBIT_head.stl
- link left_elbow: geometry visual mesh filename=package://sobit_description/mesh/stl/SOBIT_elbow v2.stl
- link left_first_arm: geometry visual mesh filename=package://sobit_description/mesh/stl/first_arm.stl
- link left_hand: geometry visual mesh filename=package://sobit_description/mesh/stl/SOBIT_hand.stl
- link left_hand_index: geometry visual mesh filename=package://sobit_description/mesh/stl/SOBIT_index.stl
- link left_hand_middle: geometry visual mesh filename=package://sobit_description/mesh/stl/SOBIT_index.stl scale=1 1 1.0588
- link left_hand_pinky: geometry visual mesh filename=package://sobit_description/mesh/stl/SOBIT_index.stl scale=1 1 0.88
- link left_hand_ring: geometry visual mesh filename=package://sobit_description/mesh/stl/SOBIT_index.stl scale=1 1 1
- link left_hand_thumb: geometry visual mesh filename=package://sobit_description/mesh/stl/SOBIT_thumb.stl
- link left_second_arm: geometry visual mesh filename=package://sobit_description/mesh/stl/SOBIT_second_arm v2.stl
- link left_shoulder: geometry visual mesh filename=package://sobit_description/mesh/stl/SOBIT_shoulder v1.stl
- link left_wheel: geometry visual mesh filename=package://sobit_description/mesh/dae/wheel.dae
- link neck: geometry visual mesh filename=package://sobit_description/mesh/stl/SOBIT_neck.stl
- link right_elbow: geometry visual mesh filename=package://sobit_description/mesh/stl/SOBIT_elbow v2.stl
- link right_first_arm: geometry visual mesh filename=package://sobit_description/mesh/stl/first_arm.stl
- link right_hand: geometry visual mesh filename=package://sobit_description/mesh/stl/SOBIT_hand_right.stl
- link right_hand_thumb: geometry visual mesh filename=package://sobit_description/mesh/stl/SOBIT_thumb_right.stl
- link right_second_arm: geometry visual mesh filename=package://sobit_description/mesh/stl/SOBIT_second_arm v2.stl
- link right_shoulder: geometry visual mesh filename=package://sobit_description/mesh/stl/SOBIT_shoulder v1.stl
- link right_wheel: geometry visual mesh filename=package://sobit_description/mesh/dae/wheel.dae

Commit message: urdf更新

File: sobit_description/robots/sobit.urdf (robot description, URDF)
Before this commit: robot sobit, 24 links, 23 joints
Links:
- added link body_cover; visual mesh filename=package://sobit_description/mesh/stl/SOBIT_body1.stl
- link left_wheel: geometry visual mesh filename=package://sobit_description/mesh/stl/wheel.stl
- link right_wheel: geometry visual mesh filename=package://sobit_description/mesh/stl/wheel.stl
Joints:
- added joint baseframe to body_cover: type fixed, parent base_frame, child body_cover, origin xyz=0 0 0.03 rpy=0 0 0
- joint lidar: origin xyz=0.2 0 0.05 rpy=0 0 3.14 -> xyz=0.305 0 0.05 rpy=0 0 3.14

File: sobit_description/robots/urdf/old_sobit.urdf (robot description, URDF)
Before this commit: robot sobit, 24 links, 23 joints
Links:
- added link body_cover; visual mesh filename=package://sobit_description/mesh/stl/body.stl

Commit message: URDFの修正とそれに伴う変更

File: sobit_description/robots/sobit.urdf (robot description, URDF)
Before this commit: robot sobit, 25 links, 24 joints
Joints:
- joint L_elbow_pitch: axis 1 0 0 -> -1 0 0; limit lower=-3.14 upper=0.3 effort=1000 velocity=0.5 -> lower=-0.3 upper=3.14 effort=1000 velocity=0.5
- joint L_elbow_yaw: limit lower=-1.571 upper=3.14 effort=1000 velocity=0.5 -> lower=-3.14 upper=1.571 effort=1000 velocity=0.5; origin xyz=0.00 0 -0.175 rpy=0 0 -1.571 -> xyz=0.00 0 -0.175 rpy=0 0 1.571
- joint L_hand_middle: axis 1 0 0 -> -1 0 0; limit lower=-1.571 upper=0 effort=1000 velocity=0.5 -> lower=-3.14 upper=0 effort=1000 velocity=0.5; origin xyz=0.02 -0.01 -0.09 rpy=0 0 0 -> xyz=-0.02 -0.01 -0.09 rpy=0 0 0
- joint L_hand_pinky: axis 1 0 0 -> -1 0 0; limit lower=-1.571 upper=0 effort=1000 velocity=0.5 -> lower=-3.14 upper=0 effort=1000 velocity=0.5; origin xyz=-0.02 -0.01 -0.09 rpy=0 0 0 -> xyz=0.02 -0.01 -0.09 rpy=0 0 0
- joint L_hand_ring: axis 1 0 0 -> -1 0 0; limit lower=-1.571 upper=0 effort=1000 velocity=0.5 -> lower=-3.14 upper=0 effort=1000 velocity=0.5
- joint L_hand_thumb: axis 0 -1 0 -> 0 1 0; origin xyz=0.04 -0.035 -0.055 rpy=0 0 0 -> xyz=-0.04 0.02 -0.055 rpy=0 0 0
- joint L_hand_wrist: axis 0 0 1 -> 0 0 -1
- joint L_shoulder_pitch: axis 0 1 0 -> 0 -1 0; limit lower=-3.14 upper=1.571 effort=1000 velocity=0.5 -> lower=-1.571 upper=3.14 effort=1000 velocity=0.5
- joint R_elbow_yaw: axis 0 0 1 -> 0 0 -1; origin xyz=0.00 0 -0.175 rpy=0 0 1.571 -> xyz=0.00 0 -0.175 rpy=0 0 -1.571
- joint R_hand_twist: limit lower=-1.571 upper=0 effort=1000 velocity=0.5 -> lower=-3.14 upper=0 effort=1000 velocity=0.5
- joint R_shoulder_pitch: axis 0 1 0 -> 0 -1 0; limit lower=-3.14 upper=1.571 effort=1000 velocity=0.5 -> lower=-1.571 upper=3.14 effort=1000 velocity=0.5
- joint R_shoulder_roll: axis 1 0 0 -> -1 0 0; limit lower=-3.14 upper=0 effort=1000 velocity=0.5 -> lower=0 upper=3.14 effort=1000 velocity=0.5
- joint left_hand_index: axis 1 0 0 -> -1 0 0; limit lower=-1.571 upper=0 effort=1000 velocity=0.5 -> lower=-3.14 upper=0 effort=1000 velocity=0.5; origin xyz=0.04 -0.01 -0.09 rpy=0 0 0 -> xyz=-0.04 -0.01 -0.09 rpy=0 0 0
- joint neck_pitch: axis 0 1 0 -> 0 -1 0
- joint neck_roll: axis 0 0 1 -> 0 0 -1
- joint neck_yaw: axis 1 0 0 -> -1 0 0
- joint right_arm_to_right_hand: origin xyz=0 -0.04 -0.17 rpy=0 0 1.571 -> xyz=0 -0.04 -0.17 rpy=0 0 -1.571

Commit message: 更新

File: sobit_description/robots/sobit.urdf (robot description, URDF)
Before this commit: robot sobit, 25 links, 24 joints
Joints:
- joint L_shoulder_roll: limit lower=0 upper=3.14 effort=1000 velocity=0.5 -> lower=0 upper=3.14 effort=1000 velocity=0.1
